Commit message: refactor: 更新 Hornet 專案的 URDF 資產模型並新增自動化測試與診斷腳本

File: Hornet/urdf/robot.urdf (robot description, URDF)
Before this commit: robot urdf, 1 links, 0 joints
Links:
- removed link hatch_2_full
- added link aileron_l, mass 0.00788323; collision mesh filename=package://assets/aileron_l.stl; visual mesh filename=package://assets/aileron_l.stl
- added link aileron_r, mass 0.00788323; collision mesh filename=package://assets/aileron_r.stl; visual mesh filename=package://assets/aileron_r.stl
- added link elevator, mass 0.0355426; collision mesh filename=package://assets/elevator.stl; visual mesh filename=package://assets/elevator.stl
- added link elevator_r, mass 0.00664075; collision mesh filename=package://assets/elevator_r.stl; visual mesh filename=package://assets/elevator_r.stl
- added link front_motor_mount_rebuild_l, mass 0.0532257; collision mesh filename=package://assets/front_motor_mount_rebuild_l.stl; collision mesh filename=package://assets/motor_2207_1300kv.stl
- added link front_motor_mount_rebuild_r, mass 0.0532257; collision mesh filename=package://assets/front_motor_mount_rebuild_r.stl; collision mesh filename=package://assets/motor_2207_1300kv.stl
- added link motor_bearing, mass 0.0119723; collision mesh filename=package://assets/motor_bearing.stl; collision mesh filename=package://assets/propellor_7040.stl
- added link motor_bearing_2, mass 0.0119723; collision mesh filename=package://assets/motor_bearing.stl; collision mesh filename=package://assets/propellor_7040.stl
- added link propellor_7040, mass 0.0119723; collision mesh filename=package://assets/motor_bearing__2.stl; collision mesh filename=package://assets/propellor_7040.stl
- added link wing1, mass 2.05076; collision mesh filename=package://assets/batt_p45b_6s2p.stl; collision mesh filename=package://assets/canopy1.stl
Joints:
- added joint ailron_L: type revolute, parent wing1, child aileron_l, origin xyz=0.27001 0.149514 0.0317166 rpy=-1.5708 -0 1.5708, axis 0 0 1, limit lower=-0.523599 upper=0.523599 effort=10 velocity=10
- added joint ailron_R: type revolute, parent wing1, child aileron_r, origin xyz=-0.27001 0.149514 0.0317166 rpy=1.5708 -0 1.5708, axis 0 0 1, limit lower=-0.523599 upper=0.523599 effort=10 velocity=10
- added joint eleveter_L: type revolute, parent wing1, child elevator, origin xyz=0.0394608 0.591475 0.0120382 rpy=4.2418e-08 1.309 -3.14159, axis 0 0 1, limit lower=-0.523599 upper=0.523599 effort=10 velocity=10
- added joint eleveter_R: type revolute, parent wing1, child elevator_r, origin xyz=-0.0394609 0.591475 0.0120382 rpy=4.2418e-08 -1.309 3.14159, axis 0 0 1, limit lower=-0.523599 upper=0.523599 effort=10 velocity=10
- added joint motor_1_CW: type revolute, parent front_motor_mount_rebuild_r, child propellor_7040, origin xyz=0 0.0245 -0.0179426 rpy=1.5708 -1.5708 0, axis 0 0 1, limit lower=-3.141592653589793 upper=3.141592653589793 effort=10 velocity=10
- added joint motor_2_CCW: type revolute, parent front_motor_mount_rebuild_l, child motor_bearing, origin xyz=-0 0.0245 0.0179426 rpy=-1.5708 -1.52993 -3.14159, axis 0 0 1, limit lower=-3.141592653589793 upper=3.141592653589793 effort=10 velocity=10
- added joint motor_3_CWW: type revolute, parent wing1, child motor_bearing_2, origin xyz=-7.13e-09 0.359799 0.0349979 rpy=3.14159 -0 -0, axis 0 0 1, limit lower=-3.141592653589793 upper=3.141592653589793 effort=10 velocity=10
- added joint tiltRotor_L: type revolute, parent wing1, child front_motor_mount_rebuild_l, origin xyz=0.231766 -0.0799765 0.0352946 rpy=1.5708 -0.0174503 1.57083, axis 0 0 1, limit lower=-0 upper=1.55334 effort=10 velocity=10
- added joint tiltRotor_R: type revolute, parent wing1, child front_motor_mount_rebuild_r, origin xyz=-0.231766 -0.0799765 0.0352946 rpy=1.5708 -0.0174503 1.57076, axis 0 0 1, limit lower=0 upper=1.55334 effort=10 velocity=10
